File: acoustic-carrier-board/acoustic-carrier-board.kicad_pcb (KiCad board)
At the start: 6 copper layers, 99 x 97 mm, 445 parts, among them IC1 ECP5-BGA256, IC1101 MT41K256M16TW-107_P, J1001 BWU.FL-IPEX1, J1002 BWU.FL-IPEX1, J1003 BWU.FL-IPEX1, J1004 BWU.FL-IPEX1, J1005 BWU.FL-IPEX1, J1006 BWU.FL-IPEX1, J1007 8P8C_Shielded, J1008 BWU.FL-IPEX1, J1009 BWU.FL-IPEX1, J1010 BWU.FL-IPEX1, J1011 BWU.FL-IPEX1, J1201 HR911130A, J201 Conn_02x06_Odd_Even, J701 Conn_02x03_Odd_Even, J702 PMOD_JTAG, J703 PMOD_SPI, J704 PMOD_GPIO, J801 TYPE-C-31-M-12, J903 Conn_02x06_Odd_Even, Q201 AO3401A, SW602 SW_Push, SW603 SW_Push, SW701 SW_Push, U1001 MS9280, U1002 THS4521IDGK, U1003 DGQ2788AEN-T1-GE4, U1004 LMV321, U1005 TL432DBZ, U1201 KSZ9031RN, U201 TPS2121RUX, U202 TLV62569DBV, U203 TLV62569DBV, U204 TLV62569DBV, U205 TLV62569DBV, U206 OPA376xxDBV, U701 W25Q128JVS, U702 W25Q128JVS, U801 USB3300-EZK, U802 LMV321, Y1201 25MHz, Y401 Crystal Oscillator, Y801 Crystal_GND24_Small

Commit message: Created production files
Parts:
- moved J201 0.45 mm to (109.0, 54.0)
Changed lines of the file:
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@@
 	(footprint "Connector_PinSocket_2.54mm:PinSocket_2x06_P2.54mm_Vertical"
 		(layer "F.Cu")
-		(at 108.58 54.16 90)
+		(at 109 54 90)
 		(descr "Through hole straight socket strip, 2x06, 2.54mm pitch, double cols (from Kicad 4.0.7), script generated")
 		(tags "Through hole socket strip THT 2x06 2.54mm double row")
@@
 			(pts
 				(xy 101.73 53.84) (xy 102.45 53.93) (xy 102.42 55) (xy 106.07 55.4) (xy 106.09 58.17) (xy 107.18 58.28)
-				(xy 122.93 58.28) (xy 122.85 55.29) (xy 107.62 55.16) (xy 106.64 52.8) (xy 101.66 52.57)
+				(xy 122.93 58.28) (xy 122.85 55.29) (xy 107.62 55.16) (xy 107.17 52.75) (xy 101.66 52.57)
 			)
 		)
@@
 		(net 1)
 		(net_name "GND")
-		(layer "F.Cu")
-		(hatch edge 0.5)
-		(priority 43)
-		(connect_pads yes
-			(clearance 0.1)
-		)
-		(min_thickness 0.25)
-		(filled_areas_thickness no)
-		(fill yes
-			(thermal_gap 0.5)
-			(thermal_bridge_width 0.5)
-		)
-		(polygon
-			(pts
-				(xy 106.64 52.8) (xy 107.62 55.16) (xy 122.85 55.29) (xy 122.85 52.67)
-			)
-		)
-	)
-	(zone
-		(net 1)
-		(net_name "GND")
 		(layers "F.Cu" "B.Cu")
 		(hatch edge 0.5)
@@
 		(layers "F.Cu" "B.Cu")
 		(hatch edge 0.5)
+		(priority 43)
+		(connect_pads yes
+			(clearance 0.1)
+		)
+		(min_thickness 0.25)
+		(filled_areas_thickness no)
+		(fill yes
+			(thermal_gap 0.5)
+			(thermal_bridge_width 0.5)
+		)
+		(polygon
+			(pts
+				(xy 107.17 52.75) (xy 107.62 55.16) (xy 122.85 55.29) (xy 122.85 52.67)
+			)
+		)
+	)
+	(zone
+		(net 1)
+		(net_name "GND")
+		(layers "F.Cu" "B.Cu")
+		(hatch edge 0.5)
 		(priority 52)
 		(connect_pads yes
@@
 			)
 		)
-	)
-	(zone
-		(net 1)
-		(net_name "GND")
-		(layer "B.Cu")
-		(hatch edge 0.5)
-		(priority 3)
-		(connect_pads no
-			(clearance 0.1)
-		)
-		(min_thickness 0.25)
-		(filled_areas_thickness no)
-		(fill yes
-			(thermal_gap 0)
-			(thermal_bridge_width 0.5)
-		)
-		(polygon
-			(pts
-				(xy 107.07 52.75) (xy 107.71 55.01) (xy 122.92 55.1) (xy 122.88 52.79) (xy 107.64 52.71)
-			)
-		)
