File: acoustic-carrier-board/acoustic-carrier-board.kicad_pcb (KiCad board)
At the start: 6 copper layers, 99 x 97 mm, 445 parts, among them IC1 ECP5-BGA256, IC1101 MT41K256M16TW-107_P, J1001 BWU.FL-IPEX1, J1002 BWU.FL-IPEX1, J1003 BWU.FL-IPEX1, J1004 BWU.FL-IPEX1, J1005 BWU.FL-IPEX1, J1006 BWU.FL-IPEX1, J1007 8P8C_Shielded, J1008 BWU.FL-IPEX1, J1009 BWU.FL-IPEX1, J1010 BWU.FL-IPEX1, J1011 BWU.FL-IPEX1, J1201 HR911130A, J201 Conn_02x06_Odd_Even, J701 Conn_02x03_Odd_Even, J702 PMOD_JTAG, J703 PMOD_SPI, J704 PMOD_GPIO, J801 TYPE-C-31-M-12, J903 Conn_02x06_Odd_Even, Q201 AO3401A, SW602 SW_Push, SW603 SW_Push, SW701 SW_Push, U1001 MS9280, U1002 THS4521IDGK, U1003 DGQ2788AEN-T1-GE4, U1004 LMV321, U1005 TL432DBZ, U1201 KSZ9031RN, U201 TPS2121RUX, U202 TLV62569DBV, U203 TLV62569DBV, U204 TLV62569DBV, U205 TLV62569DBV, U206 OPA376xxDBV, U701 W25Q128JVS, U702 W25Q128JVS, U801 USB3300-EZK, U802 LMV321, Y1201 25MHz, Y401 Crystal Oscillator, Y801 Crystal_GND24_Small

Commit message: minor changes
Connections:
- J201 pad 1: GND -> /POWER/BP_5V
- J201 pad 10: /POWER/BP_5V -> GND
- J201 pad 11: GND -> /POWER/BP_5V
- J201 pad 12: /POWER/BP_5V -> GND
- J201 pad 2: /POWER/BP_5V -> GND
- J201 pad 3: GND -> /POWER/BP_5V
- J201 pad 4: /POWER/BP_5V -> GND
- J201 pad 5: GND -> /POWER/BP_5V
- J201 pad 6: /POWER/BP_5V -> GND
- J201 pad 7: GND -> /POWER/BP_5V
- J201 pad 8: /POWER/BP_5V -> GND
- J201 pad 9: GND -> /POWER/BP_5V
Routing:
- net GND: vias 421 -> 417
Changed lines of the file:
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@@
 			)
 		)
+		(property "LPN" ""
+			(at 0 0 90)
+			(unlocked yes)
+			(layer "F.Fab")
+			(hide yes)
+			(effects
+				(font
+					(size 1 1)
+					(thickness 0.15)
+				)
+			)
+		)
+		(property "MPN" ""
+			(at 0 0 90)
+			(unlocked yes)
+			(layer "F.Fab")
+			(hide yes)
+			(effects
+				(font
+					(size 1 1)
+					(thickness 0.15)
+				)
+			)
+		)
 		(property ki_fp_filters "Connector*:*_2x??_*")
 		(sheetname "/POWER/")
@@
 			(layers "*.Cu" "*.Mask")
 			(remove_unused_layers no)
-			(net 1 "GND")
+			(net 45 "/POWER/BP_5V")
 			(pinfunction "Pin_1")
 			(pintype "passive")
@@
 			(layers "*.Cu" "*.Mask")
 			(remove_unused_layers no)
-			(net 45 "/POWER/BP_5V")
+			(net 1 "GND")
 			(pinfunction "Pin_2")
 			(pintype "passive")
@@
 			(layers "*.Cu" "*.Mask")
 			(remove_unused_layers no)
-			(net 1 "GND")
+			(net 45 "/POWER/BP_5V")
 			(pinfunction "Pin_3")
 			(pintype "passive")
@@
 			(layers "*.Cu" "*.Mask")
 			(remove_unused_layers no)
-			(net 45 "/POWER/BP_5V")
+			(net 1 "GND")
 			(pinfunction "Pin_4")
 			(pintype "passive")
@@
 			(layers "*.Cu" "*.Mask")
 			(remove_unused_layers no)
-			(net 1 "GND")
+			(net 45 "/POWER/BP_5V")
 			(pinfunction "Pin_5")
 			(pintype "passive")
@@
 			(layers "*.Cu" "*.Mask")
 			(remove_unused_layers no)
-			(net 45 "/POWER/BP_5V")
+			(net 1 "GND")
 			(pinfunction "Pin_6")
 			(pintype "passive")
@@
 			(layers "*.Cu" "*.Mask")
 			(remove_unused_layers no)
-			(net 1 "GND")
+			(net 45 "/POWER/BP_5V")
 			(pinfunction "Pin_7")
 			(pintype "passive")
@@
 			(layers "*.Cu" "*.Mask")
 			(remove_unused_layers no)
-			(net 45 "/POWER/BP_5V")
+			(net 1 "GND")
 			(pinfunction "Pin_8")
 			(pintype "passive")
@@
 			(layers "*.Cu" "*.Mask")
 			(remove_unused_layers no)
-			(net 1 "GND")
+			(net 45 "/POWER/BP_5V")
 			(pinfunction "Pin_9")
 			(pintype "passive")
@@
 			(layers "*.Cu" "*.Mask")
 			(remove_unused_layers no)
-			(net 45 "/POWER/BP_5V")
+			(net 1 "GND")
 			(pinfunction "Pin_10")
 			(pintype "passive")
@@
 			(layers "*.Cu" "*.Mask")
 			(remove_unused_layers no)
-			(net 1 "GND")
+			(net 45 "/POWER/BP_5V")
 			(pinfunction "Pin_11")
 			(pintype "passive")
@@
 			(layers "*.Cu" "*.Mask")
 			(remove_unused_layers no)
-			(net 45 "/POWER/BP_5V")
+			(net 1 "GND")
 			(pinfunction "Pin_12")
 			(pintype "passive")
@@
 	)
 	(via
-		(at 119.93 53.49)
-		(size 0.35)
-		(drill 0.2)
-		(layers "F.Cu" "B.Cu")
-		(free yes)
-		(net 1)
-	)
-	(via
 		(at 99.71 138.75)
 		(size 0.35)
@@
 	)
 	(via
-		(at 114.85 53.4)
-		(size 0.35)
-		(drill 0.2)
-		(layers "F.Cu" "B.Cu")
-		(free yes)
-		(net 1)
-	)
-	(via
 		(at 91.74 94.21)
 		(size 0.35)
@@
 	)
 	(via
-		(at 117.46 53.48)
-		(size 0.35)
-		(drill 0.2)
-		(layers "F.Cu" "B.Cu")
-		(free yes)
-		(net 1)
-	)
-	(via
 		(at 69.09 116.94)
 		(size 0.35)
@@
 	)
 	(via
-		(at 110.09 53.45)
-		(size 0.35)
-		(drill 0.2)
-		(layers "F.Cu" "B.Cu")
-		(free yes)
-		(net 1)
-	)
-	(via
 		(at 139.265 63.68)
 		(size 0.35)
@@
 	)
 	(segment
-		(start 115.565 66.3)
-		(end 126.205 55.66)
+		(start 92.55 76.05)
+		(end 92.55 78.35)
 		(width 0.1565)
 		(layer "B.Cu")
@@
 	)
 	(segment
-		(start 101.8 66.3)
-		(end 115.565 66.3)
+		(start 126.205 56.175)
+		(end 126.205 55.66)
 		(width 0.1565)
 		(layer "B.Cu")
@@
 	)
 	(segment
-		(start 92.55 76.05)
-		(end 92.55 78.35)
+		(start 116.08 66.3)
+		(end 126.205 56.175)
 		(width 0.1565)
 		(layer "B.Cu")
@@
 		(net 115)
 	)
+	(segment
+		(start 101.8 66.3)
+		(end 116.08 66.3)
+		(width 0.1565)
+		(layer "B.Cu")
+		(net 115)
+	)
 	(via
 		(at 93.3 84.25)
@@
 	)
 	(segment
-		(start 107.17 56.4)
-		(end 107.89925 55.67075)
-		(width 0.1565)
-		(layer "B.Cu")
-		(net 132)
-	)
-	(segment
-		(start 104.02075 58.76)
-		(end 105.74 58.76)
+		(start 129.825 54.77)
+		(end 130.545 55.49)
 		(width 0.1565)
 		(layer "B.Cu")
@@
 	)
 	(segment
-		(start 107.89925 55.67075)
-		(end 124.438258 55.67075)
+		(start 125.03 56.56)
+		(end 125.03 55.61)
 		(width 0.1565)
 		(layer "B.Cu")
@@
 	)
 	(segment
-		(start 129.825 54.77)
-		(end 130.545 55.49)
+		(start 105.97 60.39)
+		(end 107.09 59.27)
 		(width 0.1565)
 		(layer "B.Cu")
@@
 	)
 	(segment
-		(start 101.09 65.8)
-		(end 101.09 61.69075)
+		(start 102.39075 60.39)
+		(end 105.97 60.39)
 		(width 0.1565)
 		(layer "B.Cu")
@@
 	)
 	(segment
-		(start 125.339008 54.77)
-		(end 129.825 54.77)
+		(start 107.09 59.27)
+		(end 122.32 59.27)
 		(width 0.1565)
 		(layer "B.Cu")
@@
 	)
 	(segment
-		(start 107.17 57.33)
-		(end 107.17 56.4)
+		(start 125.87 54.77)
+		(end 129.825 54.77)
 		(width 0.1565)
 		(layer "B.Cu")
@@
 	)
 	(segment
-		(start 105.74 58.76)
-		(end 107.17 57.33)
+		(start 101.09 61.69075)
+		(end 102.39075 60.39)
 		(width 0.1565)
 		(layer "B.Cu")
@@
 	)
 	(segment
-		(start 101.09 61.69075)
-		(end 104.02075 58.76)
+		(start 101.09 65.8)
+		(end 101.09 61.69075)
 		(width 0.1565)
 		(layer "B.Cu")
@@
 	)
 	(segment
-		(start 124.438258 55.67075)
-		(end 125.339008 54.77)
+		(start 122.32 59.27)
+		(end 125.03 56.56)
 		(width 0.1565)
 		(layer "B.Cu")
@@
 	)
 	(segment
+		(start 125.03 55.61)
+		(end 125.87 54.77)
+		(width 0.1565)
+		(layer "B.Cu")
+		(net 132)
+	)
+	(segment
 		(start 57.99 110.94)
 		(end 55.71 113.22)
@@
 		(polygon
 			(pts
-				(xy 101.73 53.84) (xy 102.45 53.93) (xy 102.42 55) (xy 106.07 55.4) (xy 106.09 58.17) (xy 107.18 58.28)
-				(xy 122.93 58.28) (xy 122.85 55.29) (xy 107.62 55.16) (xy 107.17 52.75) (xy 101.66 52.57)
+				(xy 101.67 53.82) (xy 102.62 54.09) (xy 102.58 55.23) (xy 106.104688 55.29) (xy 122.964689 55.49)
+				(xy 123 52.65) (xy 101.66 52.57)
 			)
 		)
@@
 				(xy 69.6 67.3) (xy 70.1 67.7) (xy 73.7 67.4) (xy 74.6 67.226696) (xy 74.9 66.7) (xy 74.7 65.5) (xy 76.3 65.5)
 				(xy 77.1 65.1) (xy 78.3 65.2) (xy 80.8 65.2) (xy 83.1 65.8) (xy 85.9 66.4) (xy 88.4 66.9) (xy 90.9 67.3)
-				(xy 96.055937 67.803019) (xy 97.819801 67.306932) (xy 103.05 66.98) (xy 114.52 66.81) (xy 114.67 59.77)
+				(xy 96.055937 67.803019) (xy 97.819801 67.306932) (xy 103.17 66.78) (xy 114.520033 66.808483) (xy 114.67 59.77)
 				(xy 108.683296 60.197622) (xy 108.711032 65.1161) (xy 100.03 65.02) (xy 97.6 66.1) (xy 96.9 66.7)
 				(xy 95 66.8) (xy 90.8 66.4) (xy 88.4 66) (xy 85.9 65.5) (xy 84.5 65.5) (xy 83.3 65) (xy 80.8 64.4)
@@
 		(layers "F.Cu" "B.Cu")
 		(hatch edge 0.5)
-		(priority 32)
-		(connect_pads yes
-			(clearance 0.1)
-		)
-		(min_thickness 0.25)
-		(filled_areas_thickness no)
-		(fill yes
-			(thermal_gap 0.5)
-			(thermal_bridge_width 0.5)
-		)
-		(polygon
-			(pts
-				(xy 104.05 55.31) (xy 104.09 58.38) (xy 106.06 58.44) (xy 106.07 55.39)
-			)
-		)
-	)
-	(zone
-		(net 1)
-		(net_name "GND")
-		(layers "F.Cu" "B.Cu")
-		(hatch edge 0.5)
 		(priority 43)
 		(connect_pads yes
@@
 		(polygon
 			(pts
-				(xy 107.17 52.75) (xy 107.62 55.16) (xy 122.85 55.29) (xy 122.85 52.67)
+				(xy 104.17 55.25) (xy 104.169381 58.269872) (xy 123.011676 58.349444) (xy 122.964689 55.49)
 			)
 		)
